Commit message: changed gripper implementation

File: urdf/braccio_arm.urdf (robot description, URDF)
Before this commit: robot visual, 8 links, 7 joints
Links:
- removed link left_gripper
- removed link right_gripper
- added link left_gripper_link; visual mesh filename=package://ros_braccio_urdf/stl/braccio_left_gripper.stl scale=0.001 0.001 0.001
- added link right_gripper_link; visual mesh filename=package://ros_braccio_urdf/stl/braccio_right_gripper.stl scale=0.001 0.001 0.001
Joints:
- removed joint base
- removed joint elbow
- removed joint left_gripper
- removed joint right_gripper
- removed joint shoulder
- removed joint wrist_pitch
- removed joint wrist_roll
- added joint base_joint: type revolute, parent base_link, child braccio_base_link, origin xyz=0 0 0 rpy=0 0 0, axis 0 0 -1, limit lower=0.0 upper=3.1416 effort=1000.0 velocity=4.0
- added joint elbow_joint: type revolute, parent shoulder_link, child elbow_link, origin xyz=0 0 0.125 rpy=-1.5708 0 0, axis 1 0 0, limit lower=0 upper=3.1416 effort=1000.0 velocity=4.0
- added joint gripper_joint: type revolute, parent wrist_roll_link, child right_gripper_link, origin xyz=0.010 0 0.03 rpy=0 0 0, axis 0 -1 0, limit lower=0.7854 upper=1.5708 effort=1000.0 velocity=4.0
- added joint shoulder_joint: type revolute, parent braccio_base_link, child shoulder_link, origin xyz=0 -.002 0.072 rpy=-1.5708 0 0, axis 1 0 0, limit lower=0.2618 upper=2.8798 effort=1000.0 velocity=4.0
- added joint sub_gripper_joint: type revolute, parent wrist_roll_link, child left_gripper_link, origin xyz=-0.010 0 0.03 rpy=0 3.1416 0, axis 0 1 0, limit lower=1.216798176 upper=2.3559 effort=1000.0 velocity=4.0, mimic joint=gripper_joint
- added joint wrist_pitch_joint: type revolute, parent elbow_link, child wrist_pitch_link, origin xyz=0 0 0.125 rpy=-1.5708 0 0, axis 1 0 0, limit lower=0 upper=3.1416 effort=1000.0 velocity=4.0
- added joint wrist_roll_joint: type revolute, parent wrist_pitch_link, child wrist_roll_link, origin xyz=0 0.0 0.06 rpy=0 0 0, axis 0 0 -1, limit lower=0.0 upper=3.1416 effort=1000.0 velocity=4.0

Commit message: fixed gripper limits

File: urdf/braccio_arm.urdf (robot description, URDF)
Before this commit: robot visual, 8 links, 7 joints
Joints:
- joint base_joint: limit lower=0.0 upper=3.1416 effort=1000.0 velocity=4.0 -> lower=0.0 upper=3.1416 effort=1000.0 velocity=1.0
- joint elbow_joint: limit lower=0 upper=3.1416 effort=1000.0 velocity=4.0 -> lower=0 upper=3.1416 effort=1000.0 velocity=1.0
- joint gripper_joint: limit lower=0.7854 upper=1.5708 effort=1000.0 velocity=4.0 -> lower=1.217 upper=1.5708 effort=1000.0 velocity=1.0
- joint shoulder_joint: limit lower=0.2618 upper=2.8798 effort=1000.0 velocity=4.0 -> lower=0.2618 upper=2.8798 effort=1000.0 velocity=1.0
- joint sub_gripper_joint: limit lower=1.216798176 upper=2.3559 effort=1000.0 velocity=4.0 -> lower=1.5708 upper=2.7876 effort=1000.0 velocity=1.0
- joint wrist_pitch_joint: limit lower=0 upper=3.1416 effort=1000.0 velocity=4.0 -> lower=0 upper=3.1416 effort=1000.0 velocity=1.0
- joint wrist_roll_joint: limit lower=0.0 upper=3.1416 effort=1000.0 velocity=4.0 -> lower=0.0 upper=3.1416 effort=1000.0 velocity=1.0
